File: GPSMux.sch (KiCad schematic (older format))
At the start: 16 parts, among them P1 ICSP, P2 GPS1, P3 GPS2, P4 LLU, U1 CY8C27143-24PXI, U2 ADM3101EARQZ

Commit message: Updated BOM, zone settings modified, components 3d updated
Parts:
- C1, C2, C3, C4, C5, C6: symbol device:C -> GPSMux-rescue:C-device; Code 698-3251 -> (none); Manufacturer (none) -> AVX; P/N 06035C104K4T2A -> (none); Productor AVX -> (none); Provider RS -> (none); RS (none) -> 698-3251; mpn (none) -> 06035C104K4T2A
- D1: symbol device:LED -> GPSMux-rescue:LED-device; Code 778-1434 -> (none); Manufacturer (none) -> OSRAM; P/N LY Q396 -> (none); Productor OSRAM -> (none); Provider RS -> (none); RS (none) -> 778-1434; mpn (none) -> LY Q396
- P1, P2, P3: symbol conn:CONN_4 -> GPSMux-rescue:CONN_4-conn; Code 542-7113 -> (none); Manufacturer (none) -> Molex; P/N 53261-0471 -> (none); Productor Molex -> (none); Provider RS -> (none); RS (none) -> 542-7113; mpn (none) -> 53261-0471
- P4: symbol conn:CONN_3 -> GPSMux-rescue:CONN_3-conn; Code 542-7107 -> (none); Manufacturer (none) -> Molex; P/N 53261-0371 -> (none); Productor Molex -> (none); Provider RS -> (none); RS (none) -> 542-7107; mpn (none) -> 53261-0371
- R1: symbol device:R -> GPSMux-rescue:R-device; Code 678-9718 -> (none); Manufacturer (none) -> Vishay; P/N CRCW0603120RFKEA -> (none); Productor Vishay -> (none); Provider RS -> (none); RS (none) -> 678-9718; mpn (none) -> CRCW0603120RFKEA
- R2, R3: symbol device:R -> GPSMux-rescue:R-device; Manufacturer (none) -> Vishay; Provider RS -> (none); RS (none) -> 678-9670; mpn (none) -> CRCW06030000Z0EB
- U1: symbol cypress2:CY8C24123A -> GPSMux-rescue:CY8C24123A-cypress2; Code 125-4170 -> (none); Manufacturer (none) -> Cypress; P/N CY8C27143-24PXI -> (none); Productor Cypress -> (none); Provider RS -> (none); RS (none) -> 125-4170; mpn (none) -> CY8C27143-24PXI
- U2: symbol ad:ADM3101E -> GPSMux-rescue:ADM3101E-ad; Code 709-7966 -> (none); Manufacturer (none) -> Analog Devices; P/N ADM3101EARQZ -> (none); Productor Analog Devices -> (none); Provider RS -> (none); RS (none) -> 709-7966; mpn (none) -> ADM3101EARQZ
