File: PCB/GPSMux.sch (KiCad schematic (older format))
At the start: 16 parts, among them P1 ICSP, P2 GPS1, P3 GPS2, P4 LLU, U1 CY8C27143-24PXI, U2 ADM3101EARQZ

Commit message: Updated BOM
Parts:
- C1, C2, C3, C4, C5, C6: mpn 06035C104K4T2A -> 06035C104K4T2A
- D1: value LY Q396 -> LY Q396; RS 778-1434 -> 778-1434; mpn LY Q396 -> LY Q396
- P1, P2, P3: RS 542-7113 -> 542-7113
- R1: RS 678-9718 -> 678-9718; mpn CRCW0603120RFKEA -> CRCW0603120RFKEA
- U1: RS 125-4170 -> 125-4170
- U2: value ADM3101EARQZ -> ADM3101EARQZ; RS 709-7966 -> 709-7966; mpn ADM3101EARQZ -> ADM3101EARQZ
Changed lines of the file:
@@
 F 4 "Cypress" H 5225 4850 50  0001 C CNN "Manufacturer"
 F 5 "CY8C27143-24PXI" H 5225 4800 50  0001 C CNN "mpn"
-F 6 "125-4170 " H 5200 3825 50  0001 C CNN "RS"
+F 6 "125-4170" H 5200 3825 50  0001 C CNN "RS"
 	1    5200 3825
 	1    0    0    -1
@@
 P 8500 3700
 F 0 "U2" H 8500 4450 39  0000 C CNN
-F 1 "ADM3101EARQZ " H 8500 4350 39  0000 C CNN
+F 1 "ADM3101EARQZ" H 8500 4350 39  0000 C CNN
 F 2 "analog:QSOP16" H 8500 3700 50  0001 C CNN
 F 3 "" H 8500 3700 50  0001 C CNN
 F 4 "Analog Devices" H 8500 3700 50  0001 C CNN "Manufacturer"
-F 5 "ADM3101EARQZ " H 8500 3700 50  0001 C CNN "mpn"
-F 6 "709-7966 " H 8500 3700 50  0001 C CNN "RS"
+F 5 "ADM3101EARQZ" H 8500 3700 50  0001 C CNN "mpn"
+F 6 "709-7966" H 8500 3700 50  0001 C CNN "RS"
 	1    8500 3700
 	1    0    0    -1
@@
 F 4 "Molex" H 1325 2225 50  0001 C CNN "Manufacturer"
 F 5 "53261-0471" H 1325 2225 50  0001 C CNN "mpn"
-F 6 "542-7113 " H 1325 2225 50  0001 C CNN "RS"
+F 6 "542-7113" H 1325 2225 50  0001 C CNN "RS"
 	1    1325 2225
 	-1   0    0    1
@@
 F 2 "Capacitors_SMD:C_0603" H 6088 4150 30  0001 C CNN
 F 3 "" H 6050 4300 60  0000 C CNN
-F 4 "06035C104K4T2A " H 0   0   50  0001 C CNN "mpn"
+F 4 "06035C104K4T2A" H 0   0   50  0001 C CNN "mpn"
 F 5 "AVX" H 0   0   50  0001 C CNN "Manufacturer"
 F 6 "698-3251" H 6050 4300 50  0001 C CNN "RS"
@@
 F 2 "Resistors_SMD:R_0603_HandSoldering" H 4175 2500 30  0001 R CNN
 F 3 "" H 4250 2425 30  0000 C CNN
-F 4 "CRCW0603120RFKEA " H 0   0   50  0001 C CNN "mpn"
+F 4 "CRCW0603120RFKEA" H 0   0   50  0001 C CNN "mpn"
 F 5 "Vishay" H 0   0   50  0001 C CNN "Manufacturer"
-F 6 "678-9718 " H 4250 2425 50  0001 C CNN "RS"
+F 6 "678-9718" H 4250 2425 50  0001 C CNN "RS"
 	1    4250 2425
 	-1   0    0    1
@@
 P 4250 3000
 F 0 "D1" V 4175 3125 39  0000 L CNN
-F 1 " LY Q396 " V 4275 3125 39  0000 L CNN
+F 1 " LY Q396" V 4275 3125 39  0000 L CNN
 F 2 "LEDs:LED_0603_HandSoldering" V 4325 2875 39  0001 R CNN
 F 3 "" H 4250 3000 60  0001 C CNN
 F 4 "OSRAM" H 4250 3000 50  0001 C CNN "Manufacturer"
-F 5 "LY Q396 " H 4250 3000 50  0001 C CNN "mpn"
-F 6 "778-1434 " H 4250 3000 50  0001 C CNN "RS"
+F 5 "LY Q396" H 4250 3000 50  0001 C CNN "mpn"
+F 6 "778-1434" H 4250 3000 50  0001 C CNN "RS"
 	1    4250 3000
 	0    1    1    0
@@
 F 2 "Capacitors_SMD:C_0603" H 7863 4150 30  0001 C CNN
 F 3 "" H 7825 4300 60  0000 C CNN
-F 4 "06035C104K4T2A " H -50 0   50  0001 C CNN "mpn"
+F 4 "06035C104K4T2A" H -50 0   50  0001 C CNN "mpn"
 F 5 "AVX" H -50 0   50  0001 C CNN "Manufacturer"
 F 6 "698-3251" H 7825 4300 50  0001 C CNN "RS"
@@
 F 2 "Capacitors_SMD:C_0603" V 7400 3350 30  0001 C CNN
 F 3 "" H 7550 3350 60  0000 C CNN
-F 4 "06035C104K4T2A " H -50 0   50  0001 C CNN "mpn"
+F 4 "06035C104K4T2A" H -50 0   50  0001 C CNN "mpn"
 F 5 "AVX" H -50 0   50  0001 C CNN "Manufacturer"
 F 6 "698-3251" H 7550 3350 50  0001 C CNN "RS"
@@
 F 2 "Capacitors_SMD:C_0603" H 9438 3200 30  0001 C CNN
 F 3 "" H 9400 3350 60  0000 C CNN
-F 4 "06035C104K4T2A " H 50  0   50  0001 C CNN "mpn"
+F 4 "06035C104K4T2A" H 50  0   50  0001 C CNN "mpn"
 F 5 "AVX" H 50  0   50  0001 C CNN "Manufacturer"
 F 6 "698-3251" H 9400 3350 50  0001 C CNN "RS"
@@
 F 2 "Capacitors_SMD:C_0603" H 7588 3800 30  0001 C CNN
 F 3 "" H 7550 3950 60  0000 C CNN
-F 4 "06035C104K4T2A " H -50 0   50  0001 C CNN "mpn"
+F 4 "06035C104K4T2A" H -50 0   50  0001 C CNN "mpn"
 F 5 "AVX" H -50 0   50  0001 C CNN "Manufacturer"
 F 6 "698-3251" H 7550 3950 50  0001 C CNN "RS"
@@
 F 2 "Capacitors_SMD:C_0603" H 9438 3800 30  0001 C CNN
 F 3 "" H 9400 3950 60  0000 C CNN
-F 4 "06035C104K4T2A " H 50  0   50  0001 C CNN "mpn"
+F 4 "06035C104K4T2A" H 50  0   50  0001 C CNN "mpn"
 F 5 "AVX" H 50  0   50  0001 C CNN "Manufacturer"
 F 6 "698-3251" H 9400 3950 50  0001 C CNN "RS"
@@
 F 4 "Molex" H 1325 3575 50  0001 C CNN "Manufacturer"
 F 5 "53261-0471" H 1325 3575 50  0001 C CNN "mpn"
-F 6 "542-7113 " H 1325 3575 50  0001 C CNN "RS"
+F 6 "542-7113" H 1325 3575 50  0001 C CNN "RS"
 	1    1325 3575
 	-1   0    0    1
@@
 F 4 "Molex" H 1325 2900 50  0001 C CNN "Manufacturer"
 F 5 "53261-0471" H 1325 2900 50  0001 C CNN "mpn"
-F 6 "542-7113 " H 1325 2900 50  0001 C CNN "RS"
+F 6 "542-7113" H 1325 2900 50  0001 C CNN "RS"
 	1    1325 2900
 	-1   0    0    1

Commit message: Update BOM
Parts:
- C1, C2, C3, C4, C5, C6: Digikey (none) -> 478-5309-1-ND; Mouser (none) -> 581-06035C104K4
- D1: Digikey (none) -> 475-3467-1-ND; Mouser (none) -> 720-LYQ396P1Q236
- P1, P2, P3: Digikey (none) -> WM7622CT-ND; Mouser (none) -> 538-53261-0471
- P4: Digikey (none) -> WM7621CT-ND; Mouser (none) -> 538-53261-0371
- R1: Digikey (none) -> 541-120HCT-ND; Mouser (none) -> 71-CRCW0603-120-E3
- R2, R3: Digikey (none) -> 541-4013-1-ND; Mouser (none) -> 71-CRCW06030000Z0EB
- U1: Digikey (none) -> 428-1593-ND; Mouser (none) -> 727-CY8C27143-24PXI
- U2: Digikey (none) -> ADM3101EARQZ-REELCT-ND; Mouser (none) -> 584-ADM3101EARQZ
Changed lines of the file:
@@
 F 5 "CY8C27143-24PXI" H 5225 4800 50  0001 C CNN "mpn"
 F 6 "125-4170" H 5200 3825 50  0001 C CNN "RS"
+F 7 "428-1593-ND" H 5200 3825 50  0001 C CNN "Digikey"
+F 8 "727-CY8C27143-24PXI" H 5200 3825 50  0001 C CNN "Mouser"
 	1    5200 3825
 	1    0    0    -1
@@
 F 5 "ADM3101EARQZ" H 8500 3700 50  0001 C CNN "mpn"
 F 6 "709-7966" H 8500 3700 50  0001 C CNN "RS"
+F 7 "ADM3101EARQZ-REELCT-ND" H 8500 3700 50  0001 C CNN "Digikey"
+F 8 "584-ADM3101EARQZ" H 8500 3700 50  0001 C CNN "Mouser"
 	1    8500 3700
 	1    0    0    -1
@@
 F 5 "53261-0471" H 1325 2225 50  0001 C CNN "mpn"
 F 6 "542-7113" H 1325 2225 50  0001 C CNN "RS"
+F 7 "WM7622CT-ND" H 1325 2225 50  0001 C CNN "Digikey"
+F 8 "538-53261-0471" H 1325 2225 50  0001 C CNN "Mouser"
 	1    1325 2225
 	-1   0    0    1
@@
 F 5 "AVX" H 0   0   50  0001 C CNN "Manufacturer"
 F 6 "698-3251" H 6050 4300 50  0001 C CNN "RS"
+F 7 "478-5309-1-ND" H 6050 4300 50  0001 C CNN "Digikey"
+F 8 "581-06035C104K4" H 6050 4300 50  0001 C CNN "Mouser"
 	1    6050 4300
 	1    0    0    -1
@@
 F 5 "Vishay" H 0   0   50  0001 C CNN "Manufacturer"
 F 6 "678-9718" H 4250 2425 50  0001 C CNN "RS"
+F 7 "541-120HCT-ND" H 4250 2425 50  0001 C CNN "Digikey"
+F 8 "71-CRCW0603-120-E3" H 4250 2425 50  0001 C CNN "Mouser"
 	1    4250 2425
 	-1   0    0    1
@@
 F 5 "LY Q396" H 4250 3000 50  0001 C CNN "mpn"
 F 6 "778-1434" H 4250 3000 50  0001 C CNN "RS"
+F 7 "475-3467-1-ND" H 4250 3000 50  0001 C CNN "Digikey"
+F 8 "720-LYQ396P1Q236" H 4250 3000 50  0001 C CNN "Mouser"
 	1    4250 3000
 	0    1    1    0
@@
 F 5 "AVX" H -50 0   50  0001 C CNN "Manufacturer"
 F 6 "698-3251" H 7825 4300 50  0001 C CNN "RS"
+F 7 "478-5309-1-ND" H 7825 4300 50  0001 C CNN "Digikey"
+F 8 "581-06035C104K4" H 7825 4300 50  0001 C CNN "Mouser"
 	1    7825 4300
 	1    0    0    -1
@@
 F 5 "AVX" H -50 0   50  0001 C CNN "Manufacturer"
 F 6 "698-3251" H 7550 3350 50  0001 C CNN "RS"
+F 7 "478-5309-1-ND" H 7550 3350 50  0001 C CNN "Digikey"
+F 8 "581-06035C104K4" H 7550 3350 50  0001 C CNN "Mouser"
 	1    7550 3350
 	0    1    1    0
@@
 F 5 "AVX" H 50  0   50  0001 C CNN "Manufacturer"
 F 6 "698-3251" H 9400 3350 50  0001 C CNN "RS"
+F 7 "478-5309-1-ND" H 9400 3350 50  0001 C CNN "Digikey"
+F 8 "581-06035C104K4" H 9400 3350 50  0001 C CNN "Mouser"
 	1    9400 3350
 	0    -1   1    0
@@
 F 5 "AVX" H -50 0   50  0001 C CNN "Manufacturer"
 F 6 "698-3251" H 7550 3950 50  0001 C CNN "RS"
+F 7 "478-5309-1-ND" H 7550 3950 50  0001 C CNN "Digikey"
+F 8 "581-06035C104K4" H 7550 3950 50  0001 C CNN "Mouser"
 	1    7550 3950
 	0    1    1    0
@@
 F 5 "53261-0371" H 1325 4200 50  0001 C CNN "mpn"
 F 6 "542-7107" H 1325 4200 50  0001 C CNN "RS"
+F 7 "WM7621CT-ND" H 1325 4200 50  0001 C CNN "Digikey"
+F 8 "538-53261-0371" H 1325 4200 50  0001 C CNN "Mouser"
 	1    1325 4200
 	-1   0    0    1
@@
 F 5 "678-9670" H 6450 3825 50  0001 C CNN "RS"
 F 6 "CRCW06030000Z0EB" H 6450 3825 50  0001 C CNN "mpn"
+F 7 "541-4013-1-ND" H 6450 3825 50  0001 C CNN "Digikey"
+F 8 "71-CRCW06030000Z0EB" H 6450 3825 50  0001 C CNN "Mouser"
 	1    6450 3825
 	0    -1   -1   0
@@
 F 5 "AVX" H 50  0   50  0001 C CNN "Manufacturer"
 F 6 "698-3251" H 9400 3950 50  0001 C CNN "RS"
+F 7 "478-5309-1-ND" H 9400 3950 50  0001 C CNN "Digikey"
+F 8 "581-06035C104K4" H 9400 3950 50  0001 C CNN "Mouser"
 	1    9400 3950
 	0    1    1    0
@@
 F 5 "53261-0471" H 1325 3575 50  0001 C CNN "mpn"
 F 6 "542-7113" H 1325 3575 50  0001 C CNN "RS"
+F 7 "WM7622CT-ND" H 1325 3575 50  0001 C CNN "Digikey"
+F 8 "538-53261-0471" H 1325 3575 50  0001 C CNN "Mouser"
 	1    1325 3575
 	-1   0    0    1
@@
 F 5 "678-9670" H 3825 3725 50  0001 C CNN "RS"
 F 6 "CRCW06030000Z0EB" H 3825 3725 50  0001 C CNN "mpn"
+F 7 "541-4013-1-ND" H 3825 3725 50  0001 C CNN "Digikey"
+F 8 "71-CRCW06030000Z0EB" H 3825 3725 50  0001 C CNN "Mouser"
 	1    3825 3725
 	0    -1   -1   0
@@
 F 5 "53261-0471" H 1325 2900 50  0001 C CNN "mpn"
 F 6 "542-7113" H 1325 2900 50  0001 C CNN "RS"
+F 7 "WM7622CT-ND" H 1325 2900 50  0001 C CNN "Digikey"
+F 8 "538-53261-0471" H 1325 2900 50  0001 C CNN "Mouser"
 	1    1325 2900
 	-1   0    0    1
